File: PCB_EKF/PCB_EKF.kicad_sch (KiCad schematic)
At the start: 40 parts, among them J1 Load, J2 5V, J4 UART, K1 SANYOU_SRD_Form_C, K3 SANYOU_SRD_Form_C, Q1 Q_NMOS_GDS, Q2 Q_NMOS_GDS, SW1 SW_Push_SPDT, U1 MCP6002-xSN, U2 ACS712-20A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

Commit message: add firmware and change PCB
Parts:
- removed C1, C2, C3: 100nF, Capacitor_SMD:C_0805_2012Metric, symbol Device:C
- removed R1: 47k, Resistor_SMD:R_0805_2012Metric, symbol Device:R
- removed U1: MCP6002-xSN, Package_SO:SOIC-8_3.9x4.9mm_P1.27mm, symbol Amplifier_Operational:MCP6002-xSN
- removed U2: ACS712-20A, EKF:ACS712_Module, symbol ACS712_Module:ACS712_Module
- added D6, D7, D8: LED, LED_SMD:LED_0805_2012Metric_Pad1.15x1.40mm_HandSolder, symbol Device:LED
- added JP1: Jumper_2_Open, Jumper:SolderJumper-2_P1.3mm_Open_RoundedPad1.0x1.5mm, symbol Jumper:Jumper_2_Open
- added JP2: Force Control, Connector_PinHeader_2.54mm:PinHeader_1x03_P2.54mm_Vertical, symbol Jumper:Jumper_3_Open
- added R1: Shunt, Resistor_SMD:R_2512_6332Metric_Pad1.40x3.35mm_HandSolder, symbol Device:R_US
- added U1: INA226_module, EKF:INA226_module, symbol INA226_Module:INA226_module
- R2: value 100k -> R
- R3: value 1k -> R
- R4: value 10k -> R
Connections:
- net Current_Sensor is gone; now on net indikator_2: R3.1
- net 3V3: now also JP2.2 (C), U1.8 (VCC)
- net CTRL_Charge: now also U3.3 (PB14), JP2.3 (B); no longer U3.2 (PB13)
- net CTRL_Load: now also U3.2 (PB13), JP2.1 (A); no longer U3.1 (PB12)
- net GND: now also D6.1 (K), D7.1 (K), D8.1 (K), U1.7 (GND); no longer R2.2, R4.2
- net at R3.2: now also D7.2 (A); no longer R4.1
- net indikator_1: now reaches U3.11 (PB3)
- net indikator_1: now also R2.1
- net indikator_2: now reaches U3.12 (PB4)
- net indikator_3: now reaches U3.13 (PB5)
- net indikator_3: now also R4.1
- net SCL: now reaches U3.14 (PB6)
- net SCL: now also U1.5 (SCL)
- net SDA: now reaches U3.15 (PB7)
- net SDA: now also U1.6 (SDA)
- net Alert: now reaches U3.31 (PB0)
- net Alert: now also U1.4 (Alert)
- net at BT1.1 (+), SW1.2 (B), TP1.1: now also JP1.1 (A), U1.1 (IN+)
- net ADC_Current: no longer names the net of U3.24 (PA1)
- net ADC_Vbatt: no longer names the net of U3.23 (PA0)
- net PA+ renamed Shunt-
- net Shunt-: now also R1.2, U1.2 (IN-)
- net Vbatt+ renamed Vbatt
- net Vbatt: now also U1.3 (VBUS)
- new net: D6.2 (A), R2.2
- new net: D8.2 (A), R4.2
- new net Shunt+: JP1.2 (B), R1.1
Other:
- note removed: "Rasio = 0.680 Min: 2.8V⋅0.680 ≈ 1.904V. Maks: 4.2V⋅0.680 ≈ 2.857V."
- note removed: "Rasio = 0.909 Min(-10A): 1.5V⋅0.680 ≈ 1.904V. Maks(10A): 3.5V⋅0.680 ≈ 3.182V."
- moved on the sheet: BT1, D1, D2, D3, D4, J1, J2, J4, K1, K3, Q1, Q2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

Commit message: minor change silkscreen
Parts:
- removed Q1, Q2: Q_NMOS_GDS, Package_TO_SOT_SMD:SOT-23, symbol Device:Q_NMOS_GDS
- added Q1, Q3: Q_NMOS_GSD, Package_TO_SOT_SMD:SOT-23-3, symbol Device:Q_NMOS_GSD
Connections:
- net GND: now also U3.38 (GND), Q1.2 (S), Q3.2 (S)
- net at D3.1 (K), D4.2 (A), K3.2: now also Q3.3 (D)
- net at R5.2, R6.2: now also Q1.1 (G)
- net at D1.2 (A), D2.1 (K), K1.2: now also Q1.3 (D)
- net at R10.2, R9.2: now also Q3.1 (G)
Changed lines of the file:
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@@
 	(wire
 		(pts
+			(xy 59.69 92.71) (xy 59.69 96.52)
+		)
+		(stroke
+			(width 0)
+			(type default)
+		)
+	)
+	(wire
+		(pts
 			(xy 250.19 38.1) (xy 252.73 38.1)
 		)
@@
 	(wire
 		(pts
+			(xy 60.96 92.71) (xy 59.69 92.71)
+		)
+		(stroke
+			(width 0)
+			(type default)
+		)
+	)
+	(wire
+		(pts
 			(xy 233.68 100.33) (xy 233.68 106.68)
 		)
@@
 	)
 	(symbol
+		(lib_id "Device:Q_NMOS_GSD")
+		(at 241.3 118.11 0)
+		(unit 1)
+		(exclude_from_sim no)
+		(in_bom yes)
+		(on_board yes)
+		(dnp no)
+		(fields_autoplaced yes)
+		(property "Reference" "Q1"
+			(at 246.507 116.8978 0)
+			(effects
+				(font
+					(size 1.27 1.27)
+				)
+				(justify left)
+			)
+		)
+		(property "Value" "Q_NMOS_GSD"
+			(at 246.507 119.3221 0)
+			(effects
+				(font
+					(size 1.27 1.27)
+				)
+				(justify left)
+			)
+		)
+		(property "Footprint" "Package_TO_SOT_SMD:SOT-23-3"
+			(at 246.38 115.57 0)
+			(effects
+				(font
+					(size 1.27 1.27)
+				)
+				(hide yes)
+			)
+		)
+		(property "Datasheet" "~"
+			(at 241.3 118.11 0)
+			(effects
+				(font
+					(size 1.27 1.27)
+				)
+				(hide yes)
+			)
+		)
+		(property "Description" "N-MOSFET transistor, gate/source/drain"
+			(at 241.3 118.11 0)
+			(effects
+				(font
+					(size 1.27 1.27)
+				)
+				(hide yes)
+			)
+		)
+		(pin "2"
+		)
+		(pin "3"
+		)
+		(pin "1"
+		)
+		(instances
+			(project "PCB_EKF"
+				(path "/96cdbd0c-d570-41b3-b8a1-8b764a1a0da3"
+					(reference "Q1")
+					(unit 1)
+				)
+			)
+		)
+	)
+	(symbol
 		(lib_id "Device:C")
 		(at 78.74 57.15 0)
@@
 	)
 	(symbol
+		(lib_id "power:GND")
+		(at 60.96 92.71 90)
+		(unit 1)
+		(exclude_from_sim no)
+		(in_bom yes)
+		(on_board yes)
+		(dnp no)
+		(fields_autoplaced yes)
+		(property "Reference" "#PWR03"
+			(at 67.31 92.71 0)
+			(effects
+				(font
+					(size 1.27 1.27)
+				)
+				(hide yes)
+			)
+		)
+		(property "Value" "GND"
+			(at 64.135 92.71 90)
+			(effects
+				(font
+					(size 1.27 1.27)
+				)
+				(justify right)
+			)
+		)
+		(property "Footprint" ""
+			(at 60.96 92.71 0)
+			(effects
+				(font
+					(size 1.27 1.27)
+				)
+				(hide yes)
+			)
+		)
+		(property "Datasheet" ""
+			(at 60.96 92.71 0)
+			(effects
+				(font
+					(size 1.27 1.27)
+				)
+				(hide yes)
+			)
+		)
+		(property "Description" "Power symbol creates a global label with name \"GND\" , ground"
+			(at 60.96 92.71 0)
+			(effects
+				(font
+					(size 1.27 1.27)
+				)
+				(hide yes)
+			)
+		)
+		(pin "1"
+		)
+		(instances
+			(project "PCB_EKF"
+				(path "/96cdbd0c-d570-41b3-b8a1-8b764a1a0da3"
+					(reference "#PWR03")
+					(unit 1)
+				)
+			)
+		)
+	)
+	(symbol
 		(lib_id "Device:R")
 		(at 119.38 100.33 0)
@@
 	)
 	(symbol
+		(lib_id "Device:Q_NMOS_GSD")
+		(at 182.88 116.84 0)
+		(unit 1)
+		(exclude_from_sim no)
+		(in_bom yes)
+		(on_board yes)
+		(dnp no)
+		(fields_autoplaced yes)
+		(property "Reference" "Q3"
+			(at 188.087 115.6278 0)
+			(effects
+				(font
+					(size 1.27 1.27)
+				)
+				(justify left)
+			)
+		)
+		(property "Value" "Q_NMOS_GSD"
+			(at 188.087 118.0521 0)
+			(effects
+				(font
+					(size 1.27 1.27)
+				)
+				(justify left)
+			)
+		)
+		(property "Footprint" "Package_TO_SOT_SMD:SOT-23-3"
+			(at 187.96 114.3 0)
+			(effects
+				(font
+					(size 1.27 1.27)
+				)
+				(hide yes)
+			)
+		)
+		(property "Datasheet" "~"
+			(at 182.88 116.84 0)
+			(effects
+				(font
+					(size 1.27 1.27)
+				)
+				(hide yes)
+			)
+		)
+		(property "Description" "N-MOSFET transistor, gate/source/drain"
+			(at 182.88 116.84 0)
+			(effects
+				(font
+					(size 1.27 1.27)
+				)
+				(hide yes)
+			)
+		)
+		(pin "2"
+		)
+		(pin "3"
+		)
+		(pin "1"
+		)
+		(instances
+			(project ""
+				(path "/96cdbd0c-d570-41b3-b8a1-8b764a1a0da3"
+					(reference "Q3")
+					(unit 1)
+				)
+			)
+		)
+	)
+	(symbol
 		(lib_id "Device:R")
 		(at 88.9 57.15 0)
@@
 	)
 	(symbol
-		(lib_id "Device:Q_NMOS_GDS")
-		(at 182.88 116.84 0)
-		(unit 1)
-		(exclude_from_sim no)
-		(in_bom yes)
-		(on_board yes)
-		(dnp no)
-		(fields_autoplaced yes)
-		(property "Reference" "Q2"
-			(at 188.087 115.6278 0)
-			(effects
-				(font
-					(size 1.27 1.27)
-				)
-				(justify left)
-			)
-		)
-		(property "Value" "Q_NMOS_GDS"
-			(at 188.087 118.0521 0)
-			(effects
-				(font
-					(size 1.27 1.27)
-				)
-				(justify left)
-			)
-		)
-		(property "Footprint" "Package_TO_SOT_SMD:SOT-23"
-			(at 187.96 114.3 0)
-			(effects
-				(font
-					(size 1.27 1.27)
-				)
-				(hide yes)
-			)
-		)
-		(property "Datasheet" "~"
-			(at 182.88 116.84 0)
-			(effects
-				(font
-					(size 1.27 1.27)
-				)
-				(hide yes)
-			)
-		)
-		(property "Description" "N-MOSFET transistor, gate/drain/source"
-			(at 182.88 116.84 0)
-			(effects
-				(font
-					(size 1.27 1.27)
-				)
-				(hide yes)
-			)
-		)
-		(pin "2"
-		)
-		(pin "3"
-		)
-		(pin "1"
-		)
-		(instances
-			(project "PCB_EKF"
-				(path "/96cdbd0c-d570-41b3-b8a1-8b764a1a0da3"
-					(reference "Q2")
-					(unit 1)
-				)
-			)
-		)
-	)
-	(symbol
 		(lib_id "Connector:TestPoint")
 		(at 152.4 55.88 270)
@@
 					(unit 1)
 				)
-			)
-		)
-	)
-	(symbol
-		(lib_id "Device:Q_NMOS_GDS")
-		(at 241.3 118.11 0)
-		(unit 1)
-		(exclude_from_sim no)
-		(in_bom yes)
-		(on_board yes)
-		(dnp no)
-		(fields_autoplaced yes)
-		(property "Reference" "Q1"
-			(at 246.507 116.8978 0)
-			(effects
-				(font
-					(size 1.27 1.27)
-				)
-				(justify left)
-			)
-		)
-		(property "Value" "Q_NMOS_GDS"
-			(at 246.507 119.3221 0)
-			(effects
-				(font
-					(size 1.27 1.27)
-				)
-				(justify left)
-			)
-		)
-		(property "Footprint" "Package_TO_SOT_SMD:SOT-23"
-			(at 246.38 115.57 0)
-			(effects
-				(font
-					(size 1.27 1.27)
-				)
-				(hide yes)
-			)
-		)
-		(property "Datasheet" "~"
-			(at 241.3 118.11 0)
-			(effects
-				(font
-					(size 1.27 1.27)
-				)
-				(hide yes)
-			)
-		)
-		(property "Description" "N-MOSFET transistor, gate/drain/source"
-			(at 241.3 118.11 0)
-			(effects
-				(font
-					(size 1.27 1.27)
-				)
-				(hide yes)
-			)
-		)
-		(pin "2"
-		)
-		(pin "3"
-		)
-		(pin "1"
-		)
-		(instances
-			(project ""
-				(path "/96cdbd0c-d570-41b3-b8a1-8b764a1a0da3"
-					(reference "Q1")
-					(unit 1)
-				)
